File: KiCAD/FIU/fiu_board.kicad_sch (KiCad schematic)
At the start: 73 parts, among them J4 Conn_01x04_Socket, J5 Conn_01x04_Socket, J6 Conn_01x10_Socket, J7 measure wire, J9 Conn_01x10_Socket, K1 G2RL-1-H, K10 G2RL-1-H, K11 G2RL-1-H, K12 G2RL-1-H, K13 G2RL-1-H, K14 G2RL-1-H, K15 G2RL-1-H, K16 G2RL-1-H, K17 G2RL-1-H, K18 G2RL-1-H, K19 G2RL-1-H, K2 G2RL-1-H, K20 G2RL-1-H, K21 G2RL-1-H, K22 G2RL-1-H, K23 G2RL-1-H, K24 G2RL-1-H, K25 G2RL-1-H, K26 G2RL-1-H, K27 G2RL-1-H, K28 G2RL-1-H, K29 G2RL-1-H, K3 G2RL-1-H, K30 G2RL-1-H, K31 G2RL-1-H, K32 G2RL-1-H, K33 G2RL-1-H, K34 G2RL-1-H, K4 G2RL-1-H, K5 G2RL-1-H, K6 G2RL-1-H, K7 G2RL-1-H, K8 G2RL-1-H, K9 G2RL-1-H, U10 ASSR-1218, U11 ASSR-1218, U12 ASSR-1218, U13 ASSR-1218, U14 ASSR-1218, U15 ASSR-1218, U6 ASSR-1218, U7 ASSR-1218, U8 ASSR-1218, U9 ASSR-1218

Commit message: update
Parts:
- added F25, F26, F27, F28, F29, F30, F31, F32, F33, F34: 8A, symbol Device:Fuse
- added J8: Conn_01x40_Socket, symbol Connector:Conn_01x40_Socket
Connections:
- net GND: now reaches K25.A2
- net GND: now also K1.A2, K10.A2, K11.A2, K12.A2, K13.A2, K14.A2, K15.A2, K16.A2, K17.A2, K18.A2, K19.A2, K2.A2, K20.A2, K21.A2, K22.A2, K23.A2, K24.A2, K26.A2, K27.A2, K28.A2, K29.A2, K3.A2, K30.A2, K31.A2, K32.A2, K33.A2, K34.A2, K4.A2, K5.A2, K6.A2, K7.A2, K8.A2, K9.A2
- net at F18.2, U12.4: now also F31.2; no longer K15.11
- net at F20.2, U10.4: now also F29.2; no longer K28.11
- net at F21.2, U9.4: now also F28.2; no longer K23.11
- net at F8.2, U14.4: now also F33.2; no longer K30.11
- net at F17.2, U13.4: now also F32.2; no longer K21.11
- net at F23.2, U7.4: now also F26.2; no longer K13.11
- net at F22.2, U8.4: now also F27.2; no longer K18.11
- net at F6.2, U15.4: now also F34.2; no longer K33.11
- net at F24.2, U6.4: now also F25.2; no longer K7.11
- net at F19.2, U11.4: now also F30.2; no longer K9.11
- new net: F31.1, K15.11
- new net: F34.1, K33.11
- new net: F25.1, K7.11
- new net: F26.1, K13.11
- new net: F29.1, K28.11
- new net: F33.1, K30.11
- new net: F28.1, K23.11
- new net: F30.1, K9.11
- new net: F32.1, K21.11
- new net: F27.1, K18.11
- no-connect marks 11 -> 15
Other:
- moved on the sheet: K17, K19
