File: KiCAD/FIU/power.kicad_sch (KiCad schematic)
At the start: 20 parts, among them U2 lm25011my, U3 LMR10510XMFE/NOPB

Commit message: finished ethercat part
Parts:
- removed D3: D_Schottky, symbol Device:D_Schottky
- added C21, C22: 10uF 6V3, symbol Device:C
- added C23: 2.2uF 16V, symbol Device:C
- added CR1: PMEG3050EP_115, SDO_CFP5_SOD128_NEX, symbol PMEG3050EP:PMEG3050EP_115
- added CR2: STTH4R02U, SMB_STM, symbol STTH4R02U:STTH4R02U
- added D3, D4: Green, symbol Device:LED
- added L3: 2.2uH 2.3A, symbol Device:L
- added R10: 10k, symbol Device:R
- added R11, R12: 470, symbol Device:R
- added R9: 45k3, symbol Device:R
- C10, C17: value 100uF 50V -> 100nF 50V
- C15, C16: value 100uF 16V -> 4.7uF 16V
Connections:
- net GND: now also C21.2, C22.2, C23.2, CR1.2, D3.1 (K), D4.1 (K), R10.2
- net at R5.1, U2.8 (CS): now also CR2.1
- net at U3.1 (SW): now also CR1.1, L3.1
- net at U3.3 (FB): now also R10.1, R9.2
- net at C14.2, L2.1, U2.9 (SW): now also CR2.2
- new net: C21.1, C22.1, C23.1, L3.2, R11.1, R12.1, R9.1
- new net: D4.2 (A), R12.2
- new net: D3.2 (A), R11.2
Other:
- moved on the sheet: C10, C11, C12, C13, C14, C15, C16, C17, C18, C19, C20, L2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

Commit message: updated libraries
Parts:
- removed C10, C14, C17: 100nF 50V, symbol Device:C
- removed C11, C12: 4.7uF 50V, symbol Device:C
- removed C13: 22nF 50V, symbol Device:C
- removed C15, C16: 4.7uF 16V, symbol Device:C
- removed C18, C23: 2.2uF 16V, symbol Device:C
- removed C19, C20: 16uF 6V3, symbol Device:C
- removed C21, C22: 10uF 6V3, symbol Device:C
- added C11, C12, C15, C16: 4.7uF, Murata 4.7uf:CAP_GRM21_2p15X1p4X1p4_MUR, symbol Murata 4.7uf:GRM21BR61H475KE51L
- added C13: 22nF, Murata 22nF:G-155_MUR, symbol Murata 22nF:GRM155R71H223KA12D
- added C18, C52: 2.2uF, Samsung 2.2uF:CAP_CL31_SAM, symbol Samsung 2.2uF:CL31B225KBHNNNE
- added C19, C20, C21, C22: 10uF, Taiyo 10uF:CAP_UMK316BBJ106ML-T_TAY, symbol Taiyo 10uF:UMK316BBJ106ML-T
- added C24 (x3): 0.1uF, GRM155R71H104KE14J:CAP_GRM155R71H104KE14J_MUR, symbol GRM155R71H104KE14J:GRM155R71H104KE14J
- CR1: footprint SDO_CFP5_SOD128_NEX -> SDO_CFP5_SOD128_NEX:SDO_CFP5_SOD128_NEX
- CR2: footprint SMB_STM -> SMB_STM:SMB_STM
- D3, D4: footprint (none) -> LED_SMD:LED_0805_2012Metric_Pad1.15x1.40mm_HandSolder
- L2: value 10uH 1.1A -> 10uH
- L3: value 2.2uH 2.3A -> 2.2uH
- U2: footprint DGQ0010A-IPC_A -> DGQ0010A-IPC_A:DGQ0010A-IPC_A
- U3: footprint MF05A -> MF05A:MF05A
Connections:
- net +5V: now also C15.2, C16.2, C19.2, C20.2, C24.2, C52.2
- net GND: now also C11.1, C12.1, C13.1, C15.1, C16.1, C18.1, C19.1, C20.1, C21.1, C22.1, C24.1, C24.1, C52.1
- net Vin: now also C11.2, C12.2, C24.2
- net at L3.2, R11.1, R12.1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: now also C18.2, C21.2, C22.2
- net at U2.4 (SS): now also C13.2
- net at CR2.2, L2.1, U2.9 (SW): now also C24.1
- net at U2.10 (BST): now also C24.2
