File: KiCAD/FIU/EtherCAT.kicad_sch (KiCad schematic)
At the start: 0 parts

Commit message: finished ethercat part
Parts:
- added C24, C25, C26, C27, C28, C31, C32, C33, C34, C35, C36, C37, C53, C54, C55, C56, C57, C58, C59: 100nF 16V, symbol Device:C
- added C29: 1uF 16V, symbol Device:C
- added C30: 220pF 50V, symbol Device:C
- added C39, C40: 100nF 25V, symbol Device:C
- added C41, C44, C45, C46, C49, C50, C51, C52: 15pF 50V, symbol Device:C
- added C42, C43, C47, C48: 22nF 50V, symbol Device:C
- added C6: 18pF, Capacitor_SMD:C_0805_2012Metric_Pad1.18x1.45mm_HandSolder, symbol Device:C
- added C60: 2.2uF 6V3, symbol Device:C
- added D3, D4: Green, symbol Device:LED
- added J2, J3: RJ45_Wuerth_74980111211, Connector_RJ:RJ45_Wuerth_74980111211_Horizontal, symbol Connector:RJ45_Wuerth_74980111211
- added L4, L5, L6, L7: BLM18PG330SN1D, IND_BLM18_0603_MUR, symbol BLM18PG330SN1D:BLM18PG330SN1D
- added R11 (x5), R12: 470, symbol Device:R
- added R13, R16, R28, R29, R34, R35, R36, R37, R38: 4.75k, symbol Device:R
- added R17: 12k1, symbol Device:R
- added R19, R25: 10R, symbol Device:R
- added R20, R21, R22, R23, R30, R31, R32, R33: 49.9, symbol Device:R
- added U4: LAN9252/ML, QFN64_ML_MCH, symbol LAN9252/ML:LAN9252_ML
- added U5: M24C16-WMN6P, SO8N_4X5X1P27_STM, symbol M24C16:M24C16-WMN6P
- added Y1: 12Mhz, symbol Device:Crystal_GND3
Connections:
- new net: J2.12, R11.2
- new net: C44.1, J3.6 (RD+), R21.2, U4.55 (RXPA)
- new net: C50.1, J2.6 (RD+), R31.2, U4.60 (RXPB)
- new net: C41.1, J3.8 (RD-), R22.2, U4.54 (RXNA)
- new net: C6.1, U4.1 (OSCI), Y1.1
- new net: C58.1, L7.2, U4.58 (VDD33BIAS)
- new net: C37.1, R13.2, U4.11 (RST#)
- new net: D3.2 (A), R11.2
- new net: R11.1, R12.1, R16.1, U4.45 (RUNLED/E2PSIZE)
- new net: D4.2 (A), R12.2
- new net: C49.1, J2.8 (RD-), R30.2, U4.61 (RXNB)
- new net: R34.1, U5.7 (*WC)
- new net: J3.12, R11.2
- new net: C46.1, J3.3 (TD+), R23.2, U4.53 (TXPA)
- new net: J2.1, R11.2
- new net: C52.1, J2.3 (TD+), R33.2, U4.62 (TXPB)
- new net: C47.1, C48.1, J2.4 (TCT), J2.7 (RCT), R25.2
- new net: C51.1, J2.5 (TD-), R32.2, U4.63 (TXNB)
- new net: R11.2, R29.1, U4.48 (LINKACTLED0/TDO/CHIP_MODE0)
- new net: C42.1, C43.1, J3.4 (TCT), J3.7 (RCT), R19.2
- new net: C45.1, J3.5 (TD-), R20.2, U4.52 (TXNA)
- new net: R11.1, R28.1, U4.46 (LINKACTLED1/TDI/CHIP_MODE1)
- new net: R17.1, U4.57 (RBIAS)
- new net: R37.1, U4.10 (FXSDB/FXLOSB/FXSDENB), U4.8 (FXLOSEN), U4.9 (FXSDA/FXLOSA/FXSDENA)
- new net: J3.1, R11.1
- new net +1V2: C34.1, C35.1, L4.1, U4.56 (VDD12TX1), U4.59 (VDD12TX2)
- new net +3V3: C24.1, C25.1, C26.1, C27.1, C28.1, C36.1, C57.1, C59.1, C60.1, L7.1, R13.1, R35.1, R36.1, R38.2, U4.14 (VDDIO), U4.20 (VDDIO), U4.32 (VDDIO), U4.37 (VDDIO), U4.47 (VDDIO), U4.5 (VDD33), U4.7 (REG_EN), U5.8 (VCC)
- new net +3V3A: C39.1, C40.1, C55.1, C56.1, L6.1, L6.2, R19.1, R20.1, R21.1, R22.1, R23.1, U4.51 (VDD33TXRX1)
- new net +3V3B: C53.1, C54.1, L5.1, L5.2, R25.1, R30.1, R31.1, R32.1, R33.1, U4.64 (VDD33TXRX2)
- new net CS: U4.50 (D5/AD5/OUTBALID/SCS#)
- new net GND: C24.2, C25.2, C26.2, C27.2, C28.2, C29.2, C30.2, C31.2, C32.2, C33.2, C34.2, C35.2, C36.2, C37.2, C39.2, C40.2, C41.2, C42.2, C43.2, C44.2, C45.2, C46.2, C47.2, C48.2, C49.2, C50.2, C51.2, C52.2, C53.2, C54.2, C55.2, C56.2, C57.2, C58.2, C59.2, C6.2, C60.2, D3.1 (K), D4.1 (K), J2.10, J2.11, J2.2, J2.SH, J3.10, J3.11, J3.2, J3.SH, R16.2, R17.2, R28.2, R29.2, R34.2, R37.2, U4.2 (OSCO), U4.4 (OSCVSS), U4.41 (TESTMODE), U4.65 (VSS), U5.1 (NC), U5.2 (NC), U5.3 (NC), U5.4 (VSS), Y1.2, Y1.3
- new net IRQ: R38.1, U4.44 (IRQ)
- new net LAN_SYNC0: U4.34 (SYNC0/LATCH0)
- new net LAN_SYNC1: U4.18 (SYNC1/LATCH1)
- new net LED_IN: R11.1
- new net LED_OUT: R11.1
- new net MISO: U4.13 (D1/AD1/EOF/SO/SIO1)
- new net MOSI: U4.17 (D0/AD0/WD_STATE/SI/SIO0)
- new net SCK: U4.19 (D9/AD9/LATCH_IN/SCK)
- new net TCK: R35.2, U4.43 (EESCL/TCK), U5.6 (SCL)
- new net TMS: R36.2, U4.42 (EESDA/TMS), U5.5 (SDA)
- new net VDDCR: C29.1, C30.1, C31.1, C32.1, C33.1, L4.2, U4.24 (VDDCR), U4.38 (VDDCR), U4.6 (VDDCR)
- no-connect marks 0 -> 21

Commit message: updated libraries
Parts:
- removed C24, C25, C26, C27, C28, C31, C32, C33, C34, C35, C36, C37, C53, C54, C55, C56, C57, C58, C59: 100nF 16V, symbol Device:C
- removed C29: 1uF 16V, symbol Device:C
- removed C30: 220pF 50V, symbol Device:C
- removed C39, C40: 100nF 25V, symbol Device:C
- removed C41, C44, C45, C46, C49, C50, C51, C52: 15pF 50V, symbol Device:C
- removed C42, C43, C47, C48: 22nF 50V, symbol Device:C
- removed C6: 18pF, Capacitor_SMD:C_0805_2012Metric_Pad1.18x1.45mm_HandSolder, symbol Device:C
- removed C60: 2.2uF 6V3, symbol Device:C
- added C17, C24, C25, C26, C27, C28, C31, C32, C33, C34, C35, C36, C37, C39, C40, C53, C54, C55, C56, C57, C58: 0.1uF, GRM155R71H104KE14J:CAP_GRM155R71H104KE14J_MUR, symbol GRM155R71H104KE14J:GRM155R71H104KE14J
- added C29: 1uF, Murata 1uF:CAP_GRT188R61H105KE13D_MUR, symbol Murata 1uF:GRT188R61H105KE13D
- added C30: 220pF, Murata 220pF:G-188_MUR, symbol Murata 220pF:GCM1885C1H221JA16D
- added C38, C61: 18pF, Murata 15pF:G-033_MUR, symbol Murata 18pF:GRM0335C1H180JA01D
- added C41, C44, C45, C46, C49, C50, C51, C9: 15pF, Murata 15pF:G-033_MUR, symbol Murata 15pF:GRM0335C1H150JA01D
- added C52: 2.2uF, Samsung 2.2uF:CAP_CL31_SAM, symbol Samsung 2.2uF:CL31B225KBHNNNE
- added C62 (x4): 22nF, Murata 22nF:G-155_MUR, symbol Murata 22nF:GRM155R71H223KA12D
- D3, D4: footprint (none) -> LED_SMD:LED_0805_2012Metric_Pad1.15x1.40mm_HandSolder
- L4, L5, L6, L7: footprint IND_BLM18_0603_MUR -> IND_BLM18_0603_MUR':IND_BLM18_0603_MUR
- R19, R25: value 10R -> 10
- U4: footprint QFN64_ML_MCH -> QFN64_ML_MCH:QFN64_ML_MCH
- U5: footprint SO8N_4X5X1P27_STM -> SO8N_4X5X1P27_STM:SO8N_4X5X1P27_STM
- Y1: value 12Mhz -> 25Mhz
Connections:
- net +1V2: now also C34.2, C35.2
- net +3V3: now also C17.2, C24.2, C25.2, C26.2, C27.2, C28.2, C36.2, C52.2, C57.2
- net +3V3A: now also C39.2, C40.2, C55.2, C56.2
- net +3V3B: now also C53.2, C54.2
- net GND: now also C17.1, C24.1, C25.1, C26.1, C27.1, C28.1, C29.1, C30.1, C31.1, C32.1, C33.1, C34.1, C35.1, C36.1, C37.1, C38.1, C39.1, C40.1, C41.1, C44.1, C45.1, C46.1, C49.1, C50.1, C51.1, C52.1, C53.1, C54.1, C55.1, C56.1, C57.1, C58.1, C61.1, C62.1, C62.1, C62.1, C62.1, C9.1; no longer U4.2 (OSCO), Y1.2
- net VDDCR: now also C29.2, C30.2, C31.2, C32.2, C33.2
- net at J3.6 (RD+), R21.2, U4.55 (RXPA): now also C41.2
- net at J2.6 (RD+), R31.2, U4.60 (RXPB): now also C49.2
- net at J3.8 (RD-), R22.2, U4.54 (RXNA): now also C9.2
- net at U4.1 (OSCI), Y1.1: now also C38.2
- net at L7.2, U4.58 (VDD33BIAS): now also C58.2
- net at R13.2, U4.11 (RST#): now also C37.2
- net at J2.8 (RD-), R30.2, U4.61 (RXNB): now also C46.2
- net at J3.3 (TD+), R23.2, U4.53 (TXPA): now also C45.2
- net at J2.3 (TD+), R33.2, U4.62 (TXPB): now also C51.2
- net at J2.4 (TCT), J2.7 (RCT), R25.2: now also C62.2, C62.2
- net at J2.5 (TD-), R32.2, U4.63 (TXNB): now also C50.2
- net at J3.4 (TCT), J3.7 (RCT), R19.2: now also C62.2, C62.2
- net at J3.5 (TD-), R20.2, U4.52 (TXNA): now also C44.2
- new net: C61.2, U4.2 (OSCO), Y1.2

Commit message: finished front of pcb
Parts:
- removed R11 (x5), R12: 470, symbol Device:R
- removed R13, R16, R28, R29, R34, R35, R36, R37, R38: 4.75k, symbol Device:R
- removed R20, R21, R22, R23, R30, R31, R32, R33: 49.9, symbol Device:R
- removed Y1: 25Mhz, symbol Device:Crystal_GND3
- added C63, C64: 0.1uF, GRM155R71H104KE14J:CAP_GRM155R71H104KE14J_MUR, symbol GRM155R71H104KE14J:GRM155R71H104KE14J
- added R1 (x4): 470, Panasonic 470Ohm:RC0603N_PAN, symbol Panasonic 470Ohm:ERA-3AEB471V
- added R13, R16, R28, R29, R34, R35, R36, R37, R40: 4.75k, Panasonic 4.75kOhm:RC0402N_PAN-L, symbol Panasonic 4.75kOhm:ERJ-2RKF4751X
- added R20, R21, R22, R23, R30, R31, R32: 49.9, Panasonic 10kOhm:RC0402N_PAN-L, symbol Panasonic 49.9Ohm:ERJ-2RKF49R9X
- added R9: 49.9, Panasonic 49.9Ohm:RC0402N_PAN-L, symbol Panasonic 49.9Ohm:ERJ-2RKF49R9X
- added XTAL1: 25Mhz, ECS 25Mhz 18pF:ECX-32_SMDXTAL_ECS, symbol ECS 25Mhz 18pF:ECS-250-18-33-JGN-TR
- D3, D4: footprint LED_SMD:LED_0805_2012Metric_Pad1.15x1.40mm_HandSolder -> LED_SMD:LED_0603_1608Metric_Pad1.05x0.95mm_HandSolder
- R17: footprint (none) -> Resistor_SMD:R_0805_2012Metric_Pad1.20x1.40mm_HandSolder
- R19, R25: footprint (none) -> Resistor_SMD:R_0603_1608Metric_Pad0.98x0.95mm_HandSolder
Connections:
- net +3V3: now also R13.1, R34.1, R35.1, R37.1
- net +3V3A: now also R20.1, R21.1, R22.1, R9.1
- net +3V3B: now also C63.2, C64.2, R23.1, R30.1, R31.1, R32.1
- net GND: now also C63.1, C64.1, R16.2, R28.2, R29.2, R36.2, R40.2, XTAL1.2 (GND), XTAL1.4 (GND)
- net IRQ: now also R37.2
- net TCK: now also R35.2
- net TMS: now also R34.2
- net at C44.2, J3.5 (TD-), U4.52 (TXNA): now also R21.2
- net at C49.2, J2.6 (RD+), U4.60 (RXPB): now also R30.2
- net at C9.2, J3.8 (RD-), U4.54 (RXNA): now also R9.2
- net at C38.2, U4.1 (OSCI): now also XTAL1.1 (CRYSTAL)
- net at C61.2, U4.2 (OSCO): now also XTAL1.3 (CRYSTAL)
- net at D3.2 (A): now also R1.2
- net at U4.45 (RUNLED/E2PSIZE): now also R1.1, R1.1, R16.1
- net at D4.2 (A): now also R1.2
- net at C46.2, J2.8 (RD-), U4.61 (RXNB): now also R23.2
- net at C41.2, J3.6 (RD+), U4.55 (RXPA): now also R20.2
- net at U5.7 (*WC): now also R40.1
- net at J2.1: now also R1.1
- net at C51.2, J2.3 (TD+), U4.62 (TXPB): now also R32.2
- net at C50.2, J2.5 (TD-), U4.63 (TXNB): now also R31.2
- net at C37.2, U4.11 (RST#): now also R13.2
- net at U4.48 (LINKACTLED0/TDO/CHIP_MODE0): now also R1.2, R29.1
- net at U4.46 (LINKACTLED1/TDI/CHIP_MODE1): now also R1.2, R28.1
- net at C45.2, J3.3 (TD+), U4.53 (TXPA): now also R22.2
- net at U4.10 (FXSDB/FXLOSB/FXSDENB), U4.8 (FXLOSEN), U4.9 (FXSDA/FXLOSA/FXSDENA): now also R36.1
- net at J3.1: now also R1.1
- no-connect marks 21 -> 22
Other:
- moved on the sheet: C38, D3, D4
