File: KiCAD/relay_board/relay_board.kicad_sch (KiCad schematic)
At the start: 54 parts, among them J1 Conn_01x01_Socket, J10 Conn_01x01_Pin, J11 Conn_01x01_Pin, J12 Conn_01x01_Pin, J13 Conn_01x01_Pin, J14 Conn_01x01_Pin, J2 Conn_01x01_Pin, J3 Conn_01x01_Socket, J4 Conn_01x01_Pin, J5 Conn_01x01_Socket, J6 Conn_01x01_Pin, J7 Conn_01x01_Socket, J8 Conn_01x01_Pin, J9 Conn_01x01_Pin, U1 34.81-8240, U10 34.81-8240, U2 34.81-8240, U3 34.81-8240, U4 34.81-8240, U5 34.81-8240, U6 34.81-8240, U7 34.81-8240, U8 34.81-8240, U9 34.81-8240

Commit message: updated libraries
Parts:
- removed J1, J3, J5, J7: Conn_01x01_Socket, symbol Connector:Conn_01x01_Socket
- removed J10, J11, J12, J13, J14, J2, J4, J6, J8, J9: Conn_01x01_Pin, symbol Connector:Conn_01x01_Pin
- removed R1, R12, R15, R18, R21, R24, R27, R30, R6, R9: 0, symbol Device:R
- removed R10, R13, R16, R19, R2, R22, R25, R28, R4, R7: 50, symbol Device:R
- removed R11, R14, R17, R20, R23, R26, R29, R3, R5, R8: 60, symbol Device:R
- removed U1, U10, U2, U3, U4, U5, U6, U7, U8, U9: 34.81-8240, OptoDevice:Finder_34.81, symbol Relay_SolidState:34.81-8240
- added F1, F2, F3: 80A, symbol Device:Fuse
- added F10, F11, F12, F13, F14, F15, F16, F17, F18, F19, F20, F21, F22, F23, F24, F25, F26, F27, F28, F29, F30, F31, F32, F33, F34, F5, F6, F7, F8, F9: 8A, symbol Device:Fuse
- added F4: 5A, symbol Device:Fuse
- added J4, J5: Conn_01x04_Socket, symbol Connector:Conn_01x04_Socket
- added J6, J9: Conn_01x10_Socket, symbol Connector:Conn_01x10_Socket
- added J7: measure wire, symbol Connector:Conn_01x10_Socket
- added J8: Conn_01x40_Socket, symbol Connector:Conn_01x40_Socket
- added K1, K10, K11, K12, K13, K14, K15, K16, K17, K18, K19, K2, K20, K21, K22, K23, K24, K25, K26, K27, K28, K29, K3, K30, K31, K32, K33, K34, K4, K5, K6, K7, K8, K9: G2RL-1-H, Relay_THT:Relay_SPDT_Omron_G2RL-1, symbol Relay:G2RL-1-H
- added U10, U11, U12, U13, U14, U15, U6, U7, U8, U9: ASSR-1218, Package_SO:SO-4_4.4x4.3mm_P2.54mm, symbol Relay_SolidState:ASSR-1218
Connections:
- net GND: now also K1.A2, K10.A2, K11.A2, K12.A2, K13.A2, K14.A2, K15.A2, K16.A2, K17.A2, K18.A2, K19.A2, K2.A2, K20.A2, K21.A2, K22.A2, K23.A2, K24.A2, K25.A2, K26.A2, K27.A2, K28.A2, K29.A2, K3.A2, K30.A2, K31.A2, K32.A2, K33.A2, K34.A2, K4.A2, K5.A2, K6.A2, K7.A2, K8.A2, K9.A2
- new net: F27.1, K18.11
- new net: F22.2, F27.2, U8.4
- new net: K18.14, K19.11
- new net: F3.2, J5.3 (Pin_3), K11.12, K14.12, K16.12, K19.12, K24.12, K25.12, K29.12, K31.12, K34.12, K6.12
- new net: K17.11, K19.14
- new net: F20.1, J9.5 (Pin_5)
- new net: F20.2, F29.2, U10.4
- new net: F2.1, K2.12
- new net: F2.2, J5.2 (Pin_2), K10.12, K12.12, K17.12, K20.12, K22.12, K26.12, K27.12, K32.12, K4.12, K8.12
- new net: F4.1, K5.12
- new net: F4.2, J5.4 (Pin_4)
- new net: K11.14, K8.11
- new net: F1.2, J5.1 (Pin_1), K10.14, K12.14, K17.14, K20.14, K22.14, K26.14, K27.14, K32.14, K4.14, K8.14
- new net: F33.1, K30.11
- new net: K30.14, K31.11
- new net: F17.1, J9.8 (Pin_8)
- new net: F17.2, F32.2, U13.4
- new net: F32.1, K21.11
- new net: K20.11, K25.14
- new net: F25.1, K7.11
- new net: K6.11, K7.14
- new net: F10.1, J6.4 (Pin_4), J7.7 (Pin_7)
- new net: F10.2, U9.3
- new net: F28.1, K23.11
- new net: F21.2, F28.2, U9.4
- new net: K10.11, K14.14
- new net: F9.2, U8.3
- new net: K33.14, K34.11
- new net: K32.11, K34.14
- new net: F13.1, J6.7 (Pin_7), J7.4 (Pin_4)
- new net: F13.2, U12.3
- new net: K11.11, K9.14
- new net: K21.14, K25.11
- new net: F16.1, J6.10 (Pin_10), J7.1 (Pin_1)
- new net: F5.1, J6.1 (Pin_1), J7.10 (Pin_10)
- new net: F15.1, J6.9 (Pin_9), J7.2 (Pin_2)
- new net: F14.1, J6.8 (Pin_8), J7.3 (Pin_3)
- new net: F12.1, J6.6 (Pin_6), J7.5 (Pin_5)
- new net: F11.1, J6.5 (Pin_5), J7.6 (Pin_6)
- new net: F9.1, J6.3 (Pin_3), J7.8 (Pin_8)
- new net: F7.1, J6.2 (Pin_2), J7.9 (Pin_9)
- new net: K22.11, K24.14
- new net: K12.11, K16.14
- new net: F11.2, U10.3
- new net: F5.2, U6.3
- new net: F21.1, J9.4 (Pin_4)
- new net: F33.2, F8.2, U14.4
- new net: F15.2, U14.3
- new net: K4.11, K6.14
- new net: F14.2, U13.3
- new net: F12.2, U11.3
- new net: F19.2, F30.2, U11.4
- new net: F8.1, J9.9 (Pin_9)
- new net: F26.1, K13.11
- new net: F23.2, F26.2, U7.4
- new net: K13.14, K14.11
- new net: F3.1, K1.12
- new net: F24.1, J9.1 (Pin_1)
- new net: F24.2, F25.2, U6.4
- new net: K27.11, K29.14
- new net: F22.1, J9.3 (Pin_3)
- new net: F23.1, J9.2 (Pin_2)
- new net: F31.1, K15.11
- new net: K15.14, K16.11
- new net: F29.1, K28.11
- new net: K28.14, K29.11
- new net: K26.11, K31.14
- new net: F30.1, K9.11
- new net: F7.2, U7.3
- new net: F19.1, J9.6 (Pin_6)
- new net: F1.1, K3.12
- new net: K23.14, K24.11
- new net: F16.2, U15.3
- new net: F34.2, F6.2, U15.4
- new net: F6.1, J9.10 (Pin_10)
- new net: F34.1, K33.11
- new net: F18.1, J9.7 (Pin_7)
- new net: F18.2, F31.2, U12.4
- new net COM: J4.4 (Pin_4), K3.11
- new net KL15: J4.1 (Pin_1), K5.11
- new net KL30: J4.2 (Pin_2), K1.11
- new net KL31: J4.3 (Pin_3), K2.11
- no-connect marks 0 -> 15
Other:
- note added: "Interuption relays"
